File: hardware/pcb/power.kicad_sch (KiCad schematic)
At the start: 0 parts

Commit message: Capture the power sheet
All 27 components and 19 nets from power-sheet.md. ERC clean at 0 violations,
and the exported netlist diffed node-by-node against that document -- every net
matches, with ITERM the one deliberate no-connect.

Two things the capture turned up that were latent in the design:

U1 pins 10 and 11 are both OUT and both were typed power_out, so tying them --
which the datasheet requires -- was an ERC error. Retyped pin 11 as passive, the
usual idiom for duplicate power pins. The netlist is unchanged.

Local labels are sheet-qualified: the boost switching node exports as
'/power/SW', not 'SW', so the HighCurrent netclass pattern 'SW' would never have
matched it and 1.51 A peak would have routed at 0.25 mm. Pattern is now
'/power/SW'. Global labels and power symbols are unqualified and were fine.

Added project-local power symbols for VBAT, VOUT, VIN_DC and +5V_RAW, which the
stock power library does not carry.

CHG and PGOOD are captured as global rather than hierarchical labels: a
hierarchical label needs a sheet pin, and a sheet pin into an uncaptured sheet
is an ERC error rather than a promise. Recorded in power-sheet.md.

Placement is functional, not tidy -- 1.27 mm grid with labelled stubs, meant to
be dragged into shape in the GUI.
Parts:
- added BT1: 18650 protected, Battery:BatteryHolder_MPD_BH-18650-PC, symbol Device:Battery_Cell
- added C1: 10u/25V, Capacitor_SMD:C_0805_2012Metric, symbol Device:C
- added C2, C3, C4, C5: 10u, Capacitor_SMD:C_0805_2012Metric, symbol Device:C
- added C6: 22u, Capacitor_SMD:C_0805_2012Metric, symbol Device:C
- added C7: 100u, Capacitor_SMD:CP_Elec_6.3x5.4, symbol Device:C_Polarized
- added D1: SS34, Diode_SMD:D_SMA, symbol Device:D_Schottky
- added FB1: FB >=1A, Inductor_SMD:L_0805_2012Metric, symbol Device:FerriteBead
- added J1: DC in, Connector_JST:JST_XH_B2B-XH-A_1x02_P2.50mm_Vertical, symbol Connector_Generic:Conn_01x02
- added J2: Battery, remote, Connector_JST:JST_XH_B2B-XH-A_1x02_P2.50mm_Vertical, symbol Connector_Generic:Conn_01x02
- added J3: Latch switch, Connector_JST:JST_XH_B4B-XH-A_1x04_P2.50mm_Vertical, symbol Connector_Generic:Conn_01x04
- added J4: Charge LEDs, Connector_JST:JST_XH_B4B-XH-A_1x04_P2.50mm_Vertical, symbol Connector_Generic:Conn_01x04
- added L1: 1uH 4.2A, Inductor_SMD:L_Vishay_IFSC-1515AH_4x4x1.8mm, symbol Device:L
- added R1: 10k, Resistor_SMD:R_0603_1608Metric, symbol Device:R
- added R10, R9: 1k, Resistor_SMD:R_0603_1608Metric, symbol Device:R
- added R2: 1k2, Resistor_SMD:R_0603_1608Metric, symbol Device:R
- added R3: 887R 1%, Resistor_SMD:R_0603_1608Metric, symbol Device:R
- added R4: 46k4, Resistor_SMD:R_0603_1608Metric, symbol Device:R
- added R5: 0R, Resistor_SMD:R_0603_1608Metric, symbol Device:R
- added R6: 100k, Resistor_SMD:R_0603_1608Metric, symbol Device:R
- added R7: 348k 1%, Resistor_SMD:R_0603_1608Metric, symbol Device:R
- added R8: 47k5 1%, Resistor_SMD:R_0603_1608Metric, symbol Device:R
- added U1: BQ24074RGT, caryatid:BQ24074RGT_QFN-16-1EP_3x3mm_P0.5mm, symbol caryatid:BQ24074RGT
- added U2: TPS61023DRL, Package_TO_SOT_SMD:SOT-563, symbol caryatid:TPS61023DRL
Connections:
- new net +5V: C7.1, FB1.2, R5.1
- new net +5V_RAW: C6.1, FB1.1, R7.1, U2.6 (VOUT)
- new net CHG_LED: J4.2 (Pin_2), R9.1
- new net DC_IN: D1.2 (A), J1.1 (Pin_1)
- new net EN_SW: J3.2 (Pin_2), R6.1, U2.2 (EN)
- new net FB: R7.2, R8.1, U2.1 (FB)
- new net GND: BT1.2 (-), C1.2, C2.2, C3.2, C4.2, C5.2, C6.2, C7.2, J1.2 (Pin_2), J2.2 (Pin_2), J3.4 (Pin_4), J4.4 (Pin_4), R1.2, R2.2, R3.2, R4.2, R6.2, R8.2, U1.17 (EP), U1.4 (CE), U1.6 (EN1), U1.8 (VSS), U2.4 (GND)
- new net ILIM: R2.1, U1.12 (ILIM)
- new net ISET: R3.1, U1.16 (ISET)
- new net LAMP: J3.3 (Pin_3), R5.2
- new net PGOOD_LED: J4.3 (Pin_3), R10.1
- new net SW: L1.2, U2.5 (SW)
- new net TMR: R4.1, U1.14 (TMR)
- new net TS: R1.1, U1.1 (TS)
- new net VBAT: BT1.1 (+), C2.1, J2.1 (Pin_1), U1.2 (BAT), U1.3 (BAT)
- new net VIN_DC: C1.1, D1.1 (K), U1.13 (IN)
- new net VOUT: C3.1, C4.1, C5.1, J3.1 (Pin_1), J4.1 (Pin_1), L1.1, U1.10 (OUT), U1.11 (OUT), U1.5 (EN2), U2.3 (VIN)
- new net ~{CHG}: R9.2, U1.9 (~{CHG})
- new net ~{PGOOD}: R10.2, U1.7 (~{PGOOD})
- no-connect marks 0 -> 1

Commit message: Remove J2, the remote-pack connector
Nothing on the platform asked for it, and it was the last route by which a
reversed cell could reach the charger. BAT is rated -0.3 V to 5 V against a
reversed cell's -4.2 V, and there is deliberately no reverse protection because
a soldered holder cannot be wired backwards. J2 was the one exception -- a
hand-crimped loom on a keyed connector that can still be crimped wrong. With it
gone the exposure is not mitigated, it is absent: no connector on the board
reaches VBAT.

Removed surgically from power.kicad_sch by the generator's deterministic UUIDs --
symbol, both wire stubs, both power symbols -- rather than by re-running the
one-shot, which would have discarded anything done in the GUI since.

124 components, VBAT down to BT1.1, C2.1, R11.1, U1.2, U1.3.

Two things this shook out. Editing the VBAT symbol's description in one sheet's
embedded lib_symbols made it disagree with the library and with the other sheets,
which ERC reported as five lib_symbol_mismatch warnings; every sheet carries its
own copy and all of them need the same edit. And place_board.py's collision check
still split parts by is_smd(), which stopped meaning front/back when everything
moved to one face -- it has been collapsed to a single group, with
tools/check_board.py remaining the authority since it reads the board itself.

ERC 0. DRC non-ratsnest 9. All eight checks pass. Pin map unchanged.
Parts:
- removed J2: Battery, remote, Connector_JST:JST_XH_B2B-XH-A_1x02_P2.50mm_Vertical, symbol Connector_Generic:Conn_01x02
Changed lines of the file:
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@@
-	)
-	(symbol
-		(lib_id "Connector_Generic:Conn_01x02")
-		(at 250.19 62.23 0)
-		(unit 1)
-		(exclude_from_sim no)
-		(in_bom yes)
-		(on_board yes)
-		(dnp no)
-		(property "Reference" "J2"
-			(at 256.19 56.23 0)
-			(effects
-				(font
-					(size 1.27 1.27)
-				)
-			)
-		)
-		(property "Value" "Battery, remote"
-			(at 256.19 59.23 0)
-			(effects
-				(font
-					(size 1.27 1.27)
-				)
-			)
-		)
-		(property "Footprint" "Connector_JST:JST_XH_B2B-XH-A_1x02_P2.50mm_Vertical"
-			(at 250.19 62.23 0)
-			(effects
-				(font
-					(size 1.27 1.27)
-				)
-				(hide yes)
-			)
-		)
-		(property "Datasheet" "~"
-			(at 250.19 62.23 0)
-			(effects
-				(font
-					(size 1.27 1.27)
-				)
-				(hide yes)
-			)
-		)
-		(property "Description" ""
-			(at 250.19 62.23 0)
-			(effects
-				(font
-					(size 1.27 1.27)
-				)
-				(hide yes)
-			)
-		)
-		(pin "1"
-		)
-		(pin "2"
-		)
-		(instances
-			(project "caryatid"
-				(path "/49c08c53-8a29-4df2-81cf-05d7b7c47990/2a268859-e48a-4840-9d32-9349703f095d"
-					(reference "J2")
-					(unit 1)
-				)
-			)
-		)
-	)
-	(wire
-		(pts
-			(xy 245.11 62.23) (xy 240.03 62.23)
-		)
-		(stroke
-			(width 0)
-			(type default)
-		)
-	)
-	(symbol
-		(lib_id "caryatid:VBAT")
-		(at 240.03 62.23 180)
-		(unit 1)
-		(exclude_from_sim no)
-		(in_bom yes)
-		(on_board yes)
-		(dnp no)
-		(property "Reference" "#PWR"
-			(at 240.03 62.23 0)
-			(effects
-				(font
-					(size 1.27 1.27)
-				)
-				(hide yes)
-			)
-		)
-		(property "Value" "VBAT"
-			(at 240.03 65.22999999999999 0)
-			(effects
-				(font
-					(size 1.27 1.27)
-				)
-			)
-		)
-		(pin "1"
-		)
-		(instances
-			(project "caryatid"
-				(path "/49c08c53-8a29-4df2-81cf-05d7b7c47990/2a268859-e48a-4840-9d32-9349703f095d"
-					(reference "#PWR?")
-					(unit 1)
-				)
-			)
-		)
-	)
-	(wire
-		(pts
-			(xy 245.11 64.77) (xy 240.03 64.77)
-		)
-		(stroke
-			(width 0)
-			(type default)
-		)
-	)
-	(symbol
-		(lib_id "power:GND")
-		(at 240.03 64.77 180)
-		(unit 1)
-		(exclude_from_sim no)
-		(in_bom yes)
-		(on_board yes)
-		(dnp no)
-		(property "Reference" "#PWR"
-			(at 240.03 64.77 0)
-			(effects
-				(font
-					(size 1.27 1.27)
-				)
-				(hide yes)
-			)
-		)
-		(property "Value" "GND"
-			(at 240.03 67.77 0)
-			(effects
-				(font
-					(size 1.27 1.27)
-				)
-			)
-		)
-		(pin "1"
-		)
-		(instances
-			(project "caryatid"
-				(path "/49c08c53-8a29-4df2-81cf-05d7b7c47990/2a268859-e48a-4840-9d32-9349703f095d"
-					(reference "#PWR?")
-					(unit 1)
-				)
-			)
-		)
 	)
 	(symbol
