File: hardware/pcb/seed.kicad_sch (KiCad schematic)
At the start: 0 parts

Commit message: Capture the seed sheet
Both socket rows and the two measurement networks -- the A10 battery gauge and
the A11 charge-status code. 12 components.

ERC has no errors. The 33 warnings are all global_label_dangling, exactly one
per Seed pin bound for panel-io or audio, which are not captured yet: 15 D0-D14,
10 A0-A9, 4 RGB/expansion, 4 audio. The count is a checksum rather than noise --
it should reach zero when those sheets land, and any other dangling label is a
real mistake.

The pin-map cross-check the checklist asks for as a distinct pass was run by
script against pins.yaml: all 31 physical pins land on a net named after the
pin. A first attempt only covered 12 of them -- the regex matched the analog
block, whose entries carry a 'seed:' alias the digital ones do not.

Seed pin nets are global labels rather than local ones, deliberately: a local
label would export as /seed/A7 and miss the A? / A?? / AUDIO_* netclass
patterns, the same trap that caught /power/SW. A10 and A11 are global too even
though both stay on this sheet, so they land in the Analog class with the rest.

Added a project-local +3V3A power symbol. Stock has +3.3VA, which is a different
net name, and the netclass pattern is written for +3V3A.
Parts:
- added A1: 1x20 socket, caryatid:DaisySeed_Socket_A_1x20, symbol caryatid:Daisy_Seed_Socket_A
- added A2: 1x20 socket, caryatid:DaisySeed_Socket_B_1x20, symbol caryatid:Daisy_Seed_Socket_B
- added C8, C9: 10n, Capacitor_SMD:C_0603_1608Metric, symbol Device:C
- added R11, R12: 100k, Resistor_SMD:R_0603_1608Metric, symbol Device:R
- added R13, R18: 1k, Resistor_SMD:R_0603_1608Metric, symbol Device:R
- added R14, R15, R16, R17: 10k 0.1%, Resistor_SMD:R_0603_1608Metric, symbol Device:R
Connections:
- new net +3V3: A2.38 (3v3D), R14.1
- new net +3V3A: A2.21 (3v3A)
- new net +5V: A2.39 (VIN)
- new net A0: A2.22 (A0/D15)
- new net A1: A2.23 (A1/D16)
- new net A10: A2.32 (A10/D25), C8.1, R13.2
- new net A10_DIV: R11.2, R12.1, R13.1
- new net A11: A2.35 (A11/D28), C9.1, R18.2
- new net A11_DIV: R14.2, R15.1, R16.1, R18.1
- new net A2: A2.24 (A2/D17)
- new net A3: A2.25 (A3/D18)
- new net A4: A2.26 (A4/D19)
- new net A5: A2.27 (A5/D20)
- new net A6: A2.28 (A6/D21)
- new net A7: A2.29 (A7/D22)
- new net A8: A2.30 (A8/D23)
- new net A9: A2.31 (A9/D24)
- new net AUDIO_IN_L: A1.16 (AUDIO IN L)
- new net AUDIO_IN_R: A1.17 (AUDIO IN R)
- new net AUDIO_OUT_L: A1.18 (AUDIO OUT L)
- new net AUDIO_OUT_R: A1.19 (AUDIO OUT R)
- new net D0: A1.1 (D0)
- new net D1: A1.2 (D1)
- new net D10: A1.11 (D10)
- new net D11: A1.12 (D11)
- new net D12: A1.13 (D12)
- new net D13: A1.14 (D13)
- new net D14: A1.15 (D14)
- new net D2: A1.3 (D2)
- new net D26: A2.33 (D26)
- new net D27: A2.34 (D27)
- new net D29: A2.36 (D29)
- new net D3: A1.4 (D3)
- new net D30: A2.37 (D30)
- new net D4: A1.5 (D4)
- new net D5: A1.6 (D5)
- new net D6: A1.7 (D6)
- new net D7: A1.8 (D7)
- new net D8: A1.9 (D8)
- new net D9: A1.10 (D9)
- new net GND: A1.20 (AGND), A2.40 (GND), C8.2, C9.2, R12.2
- new net PGOOD_LEG: R16.2, R17.1
- new net VBAT: R11.1
- new net ~{CHG}: R15.2
- new net ~{PGOOD}: R17.2
